Commit message: convayors and new robot setup for paletizing

File: src/robots/group_a/group_a_description/config/combined_system.srdf.xacro (robot description, xacro)
@@ -4,105 +4,46 @@
 group_a_moveit_config package. The original file is located at:
     src/robots/group_a/group_a_moveit_config/config/combined_system.srdf
+    Bare frame/link names on purpose - see group_a_description/urdf/group_a_macro.xacro's
+    namespace-strategy comment. Multi-robot disambiguation is done by each robot's
+    move_group instance running in its own ROS namespace with its own private
+    robot_description_semantic parameter, not by baking a namespace into frame text.
+    Link/joint names (gp_base_link, gp_link_1..gp_link_6, gp_flange, gp_tool0) come
+    from motoman_gp70l_support/urdf/gp70l_macro.xacro's own link list, instantiated
+    with prefix="gp_" - see group_a_description/urdf/group_a_macro.xacro. The
+    disable_collisions entries below are hand-written adjacent-pair defaults (this
+    workspace has no MoveIt Setup Assistant collision-matrix run against the real
+    GP70L meshes) - re-run Setup Assistant's "Self-Collisions" step against the
+    actual collision meshes if these need tightening.
 -->
 <robot xmlns:xacro="http://ros.org/xacro" name="combined_system">
-    <!-- Ορισμός παραμέτρου prefix (κενό ως προεπιλογή) -->
-    <xacro:arg name="namespace" default="" />
-    <xacro:arg name="tf_prefix" default="" />
-    <group name="all">
-        <chain base_link="$(arg namespace)/$(arg tf_prefix)lift_base_link"
-            tip_link="$(arg namespace)/$(arg tf_prefix)ur_ft_frame" />
-    </group>
-    <group name="lift">
-        <chain base_link="$(arg namespace)/$(arg tf_prefix)lift_base_link"
-            tip_link="$(arg namespace)/$(arg tf_prefix)lift_mount" />
-    </group>
-    <group name="ur">
-        <chain base_link="$(arg namespace)/$(arg tf_prefix)ur_base_link"
-            tip_link="$(arg namespace)/$(arg tf_prefix)ur_ft_frame" />
+    <group name="manipulator">
+        <chain base_link="gp_base_link" tip_link="gp_tool0" />
     </group>
     <!--VIRTUAL
     JOINT: Purpose: this element defines a virtual joint between a robot link and an external frame
     of reference (considered fixed with respect to the robot)-->
-    <virtual_joint name="world_joint" type="fixed" parent_frame="world"
-        child_link="$(arg namespace)/$(arg tf_prefix)lift_base_link" />
+    <virtual_joint name="world_joint" type="fixed" parent_frame="world" child_link="gp_base_link" />
     <!--DISABLE
     COLLISIONS: By default it is assumed that any link of the robot could potentially come into
     collision with any other link in the robot. This tag disables collision checking between a
     specified pair of links. -->
-    <disable_collisions link1="$(arg namespace)/$(arg tf_prefix)camera_link"
-        link2="$(arg namespace)/$(arg tf_prefix)ur_wrist_1_link" reason="Never" />
-    <disable_collisions link1="$(arg namespace)/$(arg tf_prefix)camera_link"
-        link2="$(arg namespace)/$(arg tf_prefix)ur_wrist_2_link" reason="Never" />
-    <disable_collisions link1="$(arg namespace)/$(arg tf_prefix)camera_link"
-        link2="$(arg namespace)/$(arg tf_prefix)ur_wrist_3_link" reason="Adjacent" />
-    <disable_collisions link1="$(arg namespace)/$(arg tf_prefix)lift_base_link"
-        link2="$(arg namespace)/$(arg tf_prefix)lift_lower_link" reason="Adjacent" />
-    <disable_collisions link1="$(arg namespace)/$(arg tf_prefix)lift_base_link"
-        link2="$(arg namespace)/$(arg tf_prefix)lift_mount_link" reason="Never" />
-    <disable_collisions link1="$(arg namespace)/$(arg tf_prefix)lift_base_link"
-        link2="$(arg namespace)/$(arg tf_prefix)lift_plate_link" reason="Adjacent" />
-    <disable_collisions link1="$(arg namespace)/$(arg tf_prefix)lift_base_link"
-        link2="$(arg namespace)/$(arg tf_prefix)lift_upper_link" reason="Default" />
-    <disable_collisions link1="$(arg namespace)/$(arg tf_prefix)lift_base_link"
-        link2="$(arg namespace)/$(arg tf_prefix)ur_base_link_inertia" reason="Never" />
-    <disable_collisions link1="$(arg namespace)/$(arg tf_prefix)lift_base_link"
-        link2="$(arg namespace)/$(arg tf_prefix)ur_shoulder_link" reason="Never" />
-    <disable_collisions link1="$(arg namespace)/$(arg tf_prefix)lift_lower_link"
-        link2="$(arg namespace)/$(arg tf_prefix)lift_mount_link" reason="Never" />
-    <disable_collisions link1="$(arg namespace)/$(arg tf_prefix)lift_lower_link"
-        link2="$(arg namespace)/$(arg tf_prefix)lift_plate_link" reason="Never" />
-    <disable_collisions link1="$(arg namespace)/$(arg tf_prefix)lift_lower_link"
-        link2="$(arg namespace)/$(arg tf_prefix)lift_upper_link" reason="Adjacent" />
-    <disable_collisions link1="$(arg namespace)/$(arg tf_prefix)lift_lower_link"
-        link2="$(arg namespace)/$(arg tf_prefix)ur_base_link_inertia" reason="Never" />
-    <disable_collisions link1="$(arg namespace)/$(arg tf_prefix)lift_lower_link"
-        link2="$(arg namespace)/$(arg tf_prefix)ur_shoulder_link" reason="Never" />
-    <disable_collisions link1="$(arg namespace)/$(arg tf_prefix)lift_lower_link"
-        link2="$(arg namespace)/$(arg tf_prefix)ur_upper_arm_link" reason="Never" />
-    <disable_collisions link1="$(arg namespace)/$(arg tf_prefix)lift_mount_link"
-        link2="$(arg namespace)/$(arg tf_prefix)lift_plate_link" reason="Never" />
-    <disable_collisions link1="$(arg namespace)/$(arg tf_prefix)lift_mount_link"
-        link2="$(arg namespace)/$(arg tf_prefix)lift_upper_link" reason="Adjacent" />
-    <disable_collisions link1="$(arg namespace)/$(arg tf_prefix)lift_mount_link"
-        link2="$(arg namespace)/$(arg tf_prefix)ur_base_link_inertia" reason="Adjacent" />
-    <disable_collisions link1="$(arg namespace)/$(arg tf_prefix)lift_mount_link"
-        link2="$(arg namespace)/$(arg tf_prefix)ur_shoulder_link" reason="Never" />
-    <disable_collisions link1="$(arg namespace)/$(arg tf_prefix)lift_plate_link"
-        link2="$(arg namespace)/$(arg tf_prefix)lift_upper_link" reason="Never" />
-    <disable_collisions link1="$(arg namespace)/$(arg tf_prefix)lift_plate_link"
-        link2="$(arg namespace)/$(arg tf_prefix)ur_base_link_inertia" reason="Never" />
-    <disable_collisions link1="$(arg namespace)/$(arg tf_prefix)lift_plate_link"
-        link2="$(arg namespace)/$(arg tf_prefix)ur_shoulder_link" reason="Never" />
-    <disable_collisions link1="$(arg namespace)/$(arg tf_prefix)lift_plate_link"
-        link2="$(arg namespace)/$(arg tf_prefix)ur_upper_arm_link" reason="Never" />
-    <disable_collisions link1="$(arg namespace)/$(arg tf_prefix)lift_upper_link"
-        link2="$(arg namespace)/$(arg tf_prefix)ur_base_link_inertia" reason="Never" />
-    <disable_collisions link1="$(arg namespace)/$(arg tf_prefix)lift_upper_link"
-        link2="$(arg namespace)/$(arg tf_prefix)ur_shoulder_link" reason="Never" />
-    <disable_collisions link1="$(arg namespace)/$(arg tf_prefix)lift_upper_link"
-        link2="$(arg namespace)/$(arg tf_prefix)ur_upper_arm_link" reason="Never" />
-    <disable_collisions link1="$(arg namespace)/$(arg tf_prefix)lift_upper_link"
-        link2="$(arg namespace)/$(arg tf_prefix)ur_wrist_1_link" reason="Never" />
-    <disable_collisions link1="$(arg namespace)/$(arg tf_prefix)ur_base_link_inertia"
-        link2="$(arg namespace)/$(arg tf_prefix)ur_shoulder_link" reason="Adjacent" />
-    <disable_collisions link1="$(arg namespace)/$(arg tf_prefix)ur_base_link_inertia"
-        link2="$(arg namespace)/$(arg tf_prefix)ur_upper_arm_link" reason="Never" />
-    <disable_collisions link1="$(arg namespace)/$(arg tf_prefix)ur_base_link_inertia"
-        link2="$(arg namespace)/$(arg tf_prefix)ur_wrist_1_link" reason="Never" />
-    <disable_collisions link1="$(arg namespace)/$(arg tf_prefix)ur_forearm_link"
-        link2="$(arg namespace)/$(arg tf_prefix)ur_upper_arm_link" reason="Adjacent" />
-    <disable_collisions link1="$(arg namespace)/$(arg tf_prefix)ur_forearm_link"
-        link2="$(arg namespace)/$(arg tf_prefix)ur_wrist_1_link" reason="Adjacent" />
-    <disable_collisions link1="$(arg namespace)/$(arg tf_prefix)ur_shoulder_link"
-        link2="$(arg namespace)/$(arg tf_prefix)ur_upper_arm_link" reason="Adjacent" />
-    <disable_collisions link1="$(arg namespace)/$(arg tf_prefix)ur_shoulder_link"
-        link2="$(arg namespace)/$(arg tf_prefix)ur_wrist_1_link" reason="Never" />
-    <disable_collisions link1="$(arg namespace)/$(arg tf_prefix)ur_shoulder_link"
-        link2="$(arg namespace)/$(arg tf_prefix)ur_wrist_2_link" reason="Never" />
-    <disable_collisions link1="$(arg namespace)/$(arg tf_prefix)ur_wrist_1_link"
-        link2="$(arg namespace)/$(arg tf_prefix)ur_wrist_2_link" reason="Adjacent" />
-    <disable_collisions link1="$(arg namespace)/$(arg tf_prefix)ur_wrist_1_link"
-        link2="$(arg namespace)/$(arg tf_prefix)ur_wrist_3_link" reason="Never" />
-    <disable_collisions link1="$(arg namespace)/$(arg tf_prefix)ur_wrist_2_link"
-        link2="$(arg namespace)/$(arg tf_prefix)ur_wrist_3_link" reason="Adjacent" />
+    <disable_collisions link1="gp_base_link" link2="gp_link_1" reason="Adjacent" />
+    <disable_collisions link1="gp_link_1" link2="gp_link_2" reason="Adjacent" />
+    <disable_collisions link1="gp_link_2" link2="gp_link_3" reason="Adjacent" />
+    <disable_collisions link1="gp_link_3" link2="gp_link_4" reason="Adjacent" />
+    <disable_collisions link1="gp_link_4" link2="gp_link_5" reason="Adjacent" />
+    <disable_collisions link1="gp_link_5" link2="gp_link_6" reason="Adjacent" />
+    <disable_collisions link1="gp_link_6" link2="gp_flange" reason="Adjacent" />
+    <disable_collisions link1="gp_flange" link2="gp_tool0" reason="Adjacent" />
+    <disable_collisions link1="gp_link_6" link2="gp_tool0" reason="Never" />
+    <disable_collisions link1="camera_link" link2="gp_link_6" reason="Adjacent" />
+    <disable_collisions link1="camera_link" link2="gp_flange" reason="Adjacent" />
+    <disable_collisions link1="camera_link" link2="gp_tool0" reason="Adjacent" />
+    <!-- Non-adjacent but geometrically close pairs on a bent arm - kept
+         disabled to match the previous UR-based SRDF's intent (avoid
+         false-positive self-collision on the wrist/forearm links closest to
+         the tool); re-enable and let MoveIt check them if that turns out to
+         be too permissive for GP70L's actual link geometry. -->
+    <disable_collisions link1="gp_link_3" link2="gp_link_5" reason="Never" />
+    <disable_collisions link1="gp_link_4" link2="gp_link_6" reason="Never" />
 </robot>

File: src/robots/group_a/group_a_description/urdf/group_a.urdf.xacro (robot description, xacro)
@@ -5,9 +5,6 @@
   <xacro:arg name="xyz" default="0 0 0" />
   <xacro:arg name="rpy" default="0 0 0" />
-  <xacro:arg name="lift_type" default="ur_620" />
-  <xacro:arg name="ur_type" default="ur10" />
   <xacro:arg name="sim_gazebo" default="false" />
   <xacro:arg name="use_fake_hardware" default="true" />
-  <xacro:arg name="tf_prefix" default="" />
   <xacro:arg name="namespace" default="" />
   <xacro:arg name="simulation_controllers"
@@ -22,9 +19,6 @@
   <xacro:group_a_robot
     parent="$(arg parent)"
-    lift_type="$(arg lift_type)"
-    ur_type="$(arg ur_type)"
     sim_gazebo="$(arg sim_gazebo)"
     use_fake_hardware="$(arg use_fake_hardware)"
-    tf_prefix="$(arg tf_prefix)"
     namespace="$(arg namespace)"
     simulation_controllers="$(arg simulation_controllers)"
